Commit message: Added wheels tp robot urdf increased robot radiaus to 0.4 in nav2 params cleaned comments in launch file

File: urdfs/rc25.urdf (robot description, URDF)
Before this commit: robot rc25, 8 links, 7 joints
Links:
- link base_link: geometry visual box size=0.650 0.380 0.250; visual cylinder length=0.070 radius=0.090

Commit message: added tof_fc_link frame in urdf published point cloud for tof_fc; reviewed on RVIZ2 OK

File: urdfs/rc25.urdf (robot description, URDF)
Before this commit: robot rc25, 8 links, 7 joints
Links:
- added link tof_fc_link; visual cylinder length=0.030 radius=0.020
Joints:
- added joint tof_fc_joint: type fixed, parent base_link, child tof_fc_link, origin xyz=0.450 -0.080 0.300 rpy=0 0 0

Commit message: teaked tof placement added tof to voxel and obstruction

File: urdfs/rc25.urdf (robot description, URDF)
Before this commit: robot rc25, 9 links, 8 joints
Joints:
- joint tof_fc_joint: origin xyz=0.450 -0.080 0.300 rpy=0 0 0 -> xyz=0.600 0 0.130 rpy=0 0 0

Commit message: added front left and right tof sensors and  point clouds

File: urdfs/rc25.urdf (robot description, URDF)
Before this commit: robot rc25, 9 links, 8 joints
Links:
- added link tof_fl_link; visual cylinder length=0.030 radius=0.020
- added link tof_fr_link; visual cylinder length=0.030 radius=0.020
Joints:
- added joint tof_fl_joint: type fixed, parent base_link, child tof_fl_link, origin xyz=0.600 0 0.130 rpy=0 0 0.785
- added joint tof_fr_joint: type fixed, parent base_link, child tof_fr_link, origin xyz=0.600 0 0.130 rpy=0 0 -0.785

Commit message: tof-ctrl filtered out distances (=-1) when status!=5 added tof fc,fl,fr sensors to obstical layer params. increased min height to 0.1m. reduced rand=ge to 1m oer the data sheet ib bright light tof-ctrl serial port name keeps changing "Zero" <> "PiZero" - maybe when code is loaded from windows PC vs in system Linux via Pi5 urdf - lowered body height. lowered tof fc,fr,fl links. Adjusted tof_fr roll to 0.08rad so that sensor dots at ground are level and alighned with other sensors!

File: urdfs/rc25.urdf (robot description, URDF)
Before this commit: robot rc25, 11 links, 10 joints
Joints:
- joint tof_fc_joint: origin xyz=0.600 0 0.130 rpy=0 0 0 -> xyz=0.600 0 0.110 rpy=0 0 0
- joint tof_fl_joint: origin xyz=0.600 0 0.130 rpy=0 0 0.785 -> xyz=0.600 0 0.110 rpy=0 0 0.785
- joint tof_fr_joint: origin xyz=0.600 0 0.130 rpy=0 0 -0.785 -> xyz=0.600 0 0.110 rpy=0 0.08 -0.785

Commit message: urdf: added mid_link for obsticals Params: used rect footprint and mid_link. Inc inflation radius for rectangle. uncommented global cost. Allow umknown: False

File: urdfs/rc25.urdf (robot description, URDF)
Before this commit: robot rc25, 11 links, 10 joints
Links:
- added link mid_link
Joints:
- added joint mid_joint: type fixed, parent base_footprint, child mid_link, origin xyz=0.230 0 0 rpy=0 0 0

Commit message: Didi not test navigation - worked on sensors wheel node: disabled battery warning when vbat=0 nav node: cone sensors using cam, lidar, tof are  in agreement. But they are currently referenced to their sonsor location. urdf: adjusted camera frame y=-0.030 since lense is offset from mount screw

File: urdfs/rc25.urdf (robot description, URDF)
Before this commit: robot rc25, 12 links, 11 joints
Joints:
- joint oak-d-base-frame: origin xyz=0.400 0 0.315 rpy=0 0 0 -> xyz=0.400 -0.030 0.315 rpy=0 0 0

Commit message: urdf: updated after remounting sensors

File: urdfs/rc25.urdf (robot description, URDF)
Before this commit: robot rc25, 12 links, 11 joints
Joints:
- joint gps_joint: origin xyz=0.110 0 0.325 rpy=0 0 0 -> xyz=0.040 0 0.250 rpy=0 0 0
- joint imu_joint: origin xyz=0 0 0.285 rpy=0 0 0 -> xyz=0 0 0.250 rpy=0 0 0
- joint lidar_joint: origin xyz=0.220 0 0.355 rpy=0 0 0 -> xyz=0.200 0 0.320 rpy=0 0 0
- joint oak-d-base-frame: origin xyz=0.400 -0.030 0.315 rpy=0 0 0 -> xyz=0.300 0.00 0.240 rpy=0 0 0

Commit message: urdf: added rear tof sensors tof node: added rear tof sensors tof-ctrl: commented out all rear tof node code - still front sensors data are mixed up

File: urdfs/rc25.urdf (robot description, URDF)
Before this commit: robot rc25, 12 links, 11 joints
Links:
- added link tof_rc_link; visual cylinder length=0.030 radius=0.020
- added link tof_rl_link; visual cylinder length=0.030 radius=0.020
- added link tof_rr_link; visual cylinder length=0.030 radius=0.020
Joints:
- added joint tof_rc_joint: type fixed, parent base_link, child tof_rc_link, origin xyz=-0.170 0 0.110 rpy=0 0 3.1415
- added joint tof_rl_joint: type fixed, parent base_link, child tof_rl_link, origin xyz=-0.170 0 0.110 rpy=0 0 -2.356
- added joint tof_rr_joint: type fixed, parent base_link, child tof_rr_link, origin xyz=-0.170 0 0.110 rpy=0 0.08 2.356
