Commit message: Fixed TOF RR and RL positions in arduino code Changed urdf TOF RR RL sensor angle in urdf Created .bashrc_rc25 setup file moved setup script from ~/.bashrc and sourced the new file

File: urdfs/rc25.urdf (robot description, URDF)
Before this commit: robot rc25, 15 links, 14 joints
Joints:
- joint tof_rl_joint: origin xyz=-0.170 0 0.110 rpy=0 0 -2.356 -> xyz=-0.170 0 0.110 rpy=0 0 2.356
- joint tof_rr_joint: origin xyz=-0.170 0 0.110 rpy=0 0.08 2.356 -> xyz=-0.170 0 0.110 rpy=0 0.0 -2.356

Commit message: adjusted sensor locations and angles I think rear TOF needs more adjustment

File: urdfs/rc25.urdf (robot description, URDF)
Before this commit: robot rc25, 15 links, 14 joints
Joints:
- joint gps_joint: origin xyz=0.040 0 0.250 rpy=0 0 0 -> xyz=0.000 0 0.250 rpy=0 0 0
- joint imu_joint: origin xyz=0 0 0.250 rpy=0 0 0 -> xyz=0.050 0 0.250 rpy=0 0 0
- joint lidar_joint: origin xyz=0.200 0 0.320 rpy=0 0 0 -> xyz=0.180 0 0.300 rpy=0 0 0
- joint oak-d-base-frame: origin xyz=0.300 0.00 0.240 rpy=0 0 0 -> xyz=0.300 0.00 0.240 rpy=0 0 0.1
- joint tof_fc_joint: origin xyz=0.600 0 0.110 rpy=0 0 0 -> xyz=0.600 0 0.110 rpy=0.0 -0.15 0
- joint tof_fl_joint: origin xyz=0.600 0 0.110 rpy=0 0 0.785 -> xyz=0.0 0.1 0 rpy=0.1 0 0.785; parent base_link -> tof_fc_link
- joint tof_fr_joint: origin xyz=0.600 0 0.110 rpy=0 0.08 -0.785 -> xyz=0.05 -0.05 0 rpy=-0.1 0 -0.785; parent base_link -> tof_fc_link
- joint tof_rc_joint: origin xyz=-0.170 0 0.110 rpy=0 0 3.1415 -> xyz=-0.140 0 0.120 rpy=0.05 0.0 3.1415
- joint tof_rl_joint: origin xyz=-0.170 0 0.110 rpy=0 0 2.356 -> xyz=-0.120 -0.020 0.120 rpy=0.05 0.0 2.356
- joint tof_rr_joint: origin xyz=-0.170 0 0.110 rpy=0 0.0 -2.356 -> xyz=-0.120 0.020 0.120 rpy=-0.1 0.0 -2.356

Commit message: TOF front sensors calibrated on flat wall ~1M dist

File: urdfs/rc25.urdf (robot description, URDF)
Before this commit: robot rc25, 15 links, 14 joints
Joints:
- joint tof_fc_joint: origin xyz=0.600 0 0.110 rpy=0.0 -0.15 0 -> xyz=0.650 0 0.09 rpy=0.0 -0.15 0.02
- joint tof_fl_joint: origin xyz=0.0 0.1 0 rpy=0.1 0 0.785 -> xyz=-0.03 0.01 0.02 rpy=0.05 0 0.75
- joint tof_fr_joint: origin xyz=0.05 -0.05 0 rpy=-0.1 0 -0.785 -> xyz=0 -0.01 0.01 rpy=-0.05 0 -0.75

Commit message: rear TOF calibrated with flat wall

File: urdfs/rc25.urdf (robot description, URDF)
Before this commit: robot rc25, 15 links, 14 joints
Joints:
- joint tof_rc_joint: origin xyz=-0.140 0 0.120 rpy=0.05 0.0 3.1415 -> xyz=-0.160 0 0.120 rpy=0.0 -0.02 3.15
- joint tof_rl_joint: origin xyz=-0.120 -0.020 0.120 rpy=0.05 0.0 2.356 -> xyz=-0.02 -0.01 0 rpy=0.0 0.0 -0.75; parent base_link -> tof_rc_link
- joint tof_rr_joint: origin xyz=-0.120 0.020 0.120 rpy=-0.1 0.0 -2.356 -> xyz=-0.01 0.02 0 rpy=-0.0 0.0 0.75; parent base_link -> tof_rc_link

Commit message: added alias foxbridge to .bashrc_rc25 added median-5 filter to imu roll,pitch,yaw reversed imu roll and pitch to compensate for imu mounting inverted imu pitch so that Rviz showed the tilt properly enabled efks 3d mode to support roll and pitch Used imu roll,pithch,yaw data in efks enabled efk_local imu relative mode to initialize orientation to zero urdf placed imu and gps at proper X location

File: urdfs/rc25.urdf (robot description, URDF)
Before this commit: robot rc25, 15 links, 14 joints
Joints:
- joint gps_joint: origin xyz=0.000 0 0.250 rpy=0 0 0 -> xyz=0.040 0 0.250 rpy=0 0 0
- joint imu_joint: origin xyz=0.050 0 0.250 rpy=0 0 0 -> xyz=0.010 0 0.250 rpy=0 0 0

Commit message: adjusted oak camera and lidar rpy-z to align and center the cone detection fom both sensors the front TOF sensors are already adjusted and detect cone as centered and aligned with the lidar and camera

File: urdfs/rc25.urdf (robot description, URDF)
Before this commit: robot rc25, 15 links, 14 joints
Joints:
- joint lidar_joint: origin xyz=0.180 0 0.300 rpy=0 0 0 -> xyz=0.180 0 0.300 rpy=0 0 -0.025
- joint oak-d-base-frame: origin xyz=0.300 0.00 0.240 rpy=0 0 0.1 -> xyz=0.340 0.00 0.240 rpy=0 0 0.05
