File: support/rc26_PowerSubsystem/rc26_PowerSubsystem.kicad_sch (KiCad schematic)
At the start: 6 parts, among them J1 12V DC

Commit message: doc update
Other:
- note removed: "DROK Buck Converter 12v to 5v with USB Type C, 24V to 12V Step Down Converter Adjustable DC Voltage Regulator 8.2V-32V to 3V-20V 4.8A Volt Transformer Power Supply for Type C Charger Fast Charging"
